File: robot.kicad_pcb (KiCad board)
At the start: 4 copper layers, 132 x 60.2 mm, 168 parts, among them J1 USB_C_Receptacle_USB2.0_16P, J2 Batt-Cell Connector, J3 Batt Connector, J4 DVR FOUT, J6 DRV BOUT, J7 UART, J8 I2C, J9 5way Tracing, Q1 AO3400A, Q2 AO3400A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

Commit message: Add gerber file
Parts:
- added J10: 5V, Connector_PinHeader_2.54mm:PinHeader_1x02_P2.54mm_Vertical, F.Cu at (187.1, 58.6)
- added J5: 3.3V, Connector_PinHeader_2.54mm:PinHeader_1x02_P2.54mm_Vertical, F.Cu at (194.0, 58.6)
- moved J7 0.12 mm to (251.3, 95.6)
Routing:
- net +5V: track 17.4 -> 28.2 mm, vias 5 -> 10
- net /Cell2: track 77.7 -> 81.0 mm
- net +BATT: track 94.7 -> 91.4 mm, vias 10 -> 15
- net GND1: track 92.2 -> 94.0 mm
- net +3.3V: track 61.5 -> 62.4 mm, vias 16 -> 20
- net /ESP32-C6-mini/F_BIN1: track 102.5 -> 101.9 mm
- net GND: track 172.0 -> 171.7 mm, vias 121 -> 129
- added copper zone on F.Cu, net +3.3V
- added copper zone on F.Cu, net +5V
- added copper zone on F.Cu, net +BATT
Other:
- board text added: "05/26 Thomas More IOT Malik B / Vladislav V"
- board text added: "5V"
- board text added: "CP"
- board text added: "Cell1"
- board text added: "Cell2"
- board text added: "DATA"
- board text added: "DIN"
- board text added: "DIN_EN"
- board text added: "DM"
- board text added: "DP"
- board text added: "LD"
- board text added: "RXD0"
- board text added: "TXD0"
- board text added: "ULED"
